Commit message: updated relative paths in URDF

File: urdf/Paucibot.urdf (robot description, URDF)
Before this commit: robot Paucibot, 11 links, 10 joints
Links:
- link BaseLink: geometry collision cylinder length=0.0055 radius=0.075; visual mesh filename=$(rospack find paucibot)/meshes/stl/Circle.004.stl scale=0.075 0.075 0.06329
- link Holder1_link: geometry collision box size=0.0509 0.04 0.0309; visual mesh filename=$(rospack find paucibot)/meshes/stl/Cube.010.stl scale=0.95238 0.7619 0.03429
- link Holder2_link: geometry collision box size=0.0509 0.04 0.0309; visual mesh filename=$(rospack find paucibot)/meshes/stl/Cube.009.stl scale=0.95238 0.7619 0.03429
- link Motor1_link: geometry collision cylinder length=0.06216 radius=0.018; visual mesh filename=$(rospack find paucibot)/meshes/stl/Cylinder.stl scale=1.0 1.0 1.0
- link Motor2_link: geometry collision cylinder length=0.06262 radius=0.018; visual mesh filename=$(rospack find paucibot)/meshes/stl/Cylinder.001.stl scale=1.0 1.0 1.0
- link UpperLink: geometry collision cylinder length=0.0055 radius=0.075; visual mesh filename=$(rospack find paucibot)/meshes/stl/Circle.003.stl scale=0.075 0.075 0.06329
- link wheel1_link: geometry collision cylinder length=0.03798 radius=0.043; visual mesh filename=$(rospack find paucibot)/meshes/stl/Torus.stl scale=0.81132 0.81132 1.89758
- link wheel2_link: geometry collision cylinder length=0.03798 radius=0.043; visual mesh filename=$(rospack find paucibot)/meshes/stl/Torus.002.stl scale=0.81132 0.81132 1.89758

Commit message: Fixed relative paths

File: urdf/Paucibot.urdf (robot description, URDF)
Before this commit: robot Paucibot, 11 links, 10 joints
Links:
- link BaseLink: geometry collision cylinder length=0.0055 radius=0.075; visual mesh filename=package://paucibot/meshes/stl/Circle.004.stl scale=0.075 0.075 0.06329
- link Holder1_link: geometry collision box size=0.0509 0.04 0.0309; visual mesh filename=package://paucibot/meshes/stl/Cube.010.stl scale=0.95238 0.7619 0.03429
- link Holder2_link: geometry collision box size=0.0509 0.04 0.0309; visual mesh filename=package://paucibot/meshes/stl/Cube.009.stl scale=0.95238 0.7619 0.03429
- link Motor1_link: geometry collision cylinder length=0.06216 radius=0.018; visual mesh filename=package://paucibot/meshes/stl/Cylinder.stl scale=1.0 1.0 1.0
- link Motor2_link: geometry collision cylinder length=0.06262 radius=0.018; visual mesh filename=package://paucibot/meshes/stl/Cylinder.001.stl scale=1.0 1.0 1.0
- link UpperLink: geometry collision cylinder length=0.0055 radius=0.075; visual mesh filename=package://paucibot/meshes/stl/Circle.003.stl scale=0.075 0.075 0.06329
- link wheel1_link: geometry collision cylinder length=0.03798 radius=0.043; visual mesh filename=package://paucibot/meshes/stl/Torus.stl scale=0.81132 0.81132 1.89758
- link wheel2_link: geometry collision cylinder length=0.03798 radius=0.043; visual mesh filename=package://paucibot/meshes/stl/Torus.002.stl scale=0.81132 0.81132 1.89758
